File: 60.kicad_pcb (KiCad board)
At the start: 2 copper layers, 285 x 94.6 mm, 154 parts, among them K1 KEYSW, K10 KEYSW, K11 KEYSW, K12 KEYSW, K13 KEYSW, K14 KEYSW, K15 KEYSW, K16 KEYSW, K17 KEYSW, K18 KEYSW, K19 KEYSW, K2 KEYSW, K20 KEYSW, K21 KEYSW, K22 KEYSW, K23 KEYSW, K24 KEYSW, K25 KEYSW, K26 KEYSW, K27 KEYSW, K28 KEYSW, K29 KEYSW, K3 KEYSW, K30 KEYSW, K31 KEYSW, K32 KEYSW, K33 KEYSW, K34 KEYSW, K35 KEYSW, K36 KEYSW, K37 KEYSW, K38 KEYSW, K39 KEYSW, K4 KEYSW, K40 KEYSW, K41 KEYSW, K42 KEYSW, K43 KEYSW, K44 KEYSW, K45 KEYSW, K46 KEYSW, K47 KEYSW, K48 KEYSW, K49 KEYSW, K5 KEYSW, K50 KEYSW, K51 KEYSW, K52 KEYSW, K53 KEYSW, K54 KEYSW, K55 KEYSW, K56 KEYSW, K57 KEYSW, K58 KEYSW, K59 KEYSW, K6 KEYSW, K60 KEYSW, K61 KEYSW, K62 KEYSW, K63 KEYSW, K64 KEYSW, K65 KEYSW, K66 KEYSW, K67 KEYSW, K68 KEYSW, K69 KEYSW, K7 KEYSW, K70 KEYSW, K71 KEYSW, K72 KEYSW, K73 KEYSW, K74 KEYSW, K75 KEYSW, K76 KEYSW, K77 KEYSW, K78 KEYSW, K79 KEYSW, K8 KEYSW, K80 KEYSW, K81 KEYSW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

Commit message: pre-diode swap
Parts:
- added BT1: Battery, Battery_Holders:Keystone_1058_1x2032-CoinCell, B.Cu at (223.8, 57.0)
- added C1: 0.1u, Capacitors_SMD:C_0805_HandSoldering, B.Cu at (35.8, 68.0)
- added C2: 0.1u, Capacitors_SMD:C_0805_HandSoldering, B.Cu at (31.2, 55.5)
- added C3: 0.1u, Capacitors_SMD:C_0805_HandSoldering, B.Cu at (42.8, 47.1)
- added C4: 0.1u, Capacitors_SMD:C_0805_HandSoldering, B.Cu at (51.2, 54.7)
- added C5: 1u, Capacitors_SMD:C_0805_HandSoldering, B.Cu at (62.5, 44.2)
- added D67: D_Schottky_x2_KCom_AAK, TO_SOT_Packages_SMD:SOT-23_Handsoldering, B.Cu at (62.0, 47.2)
- added IC1: ATXMEGA32A4U-A, Housings_QFP:TQFP-44_10x10mm_Pitch0.8mm, B.Cu at (41.8, 57.2)
- added P1: CONN_01X01, Connectors_TestPoints:Test_Point_Pad_2.0x2.0mm, B.Cu at (50.0, 51.7)
- added R1: 10k, Resistors_SMD:R_0805_HandSoldering, B.Cu at (33.3, 78.6)
- added R2: 22, Resistors_SMD:R_0805_HandSoldering, B.Cu at (23.8, 46.8)
- added R3: 22, Resistors_SMD:R_0805_HandSoldering, B.Cu at (25.8, 46.8)
- added R4: 100k, Resistors_SMD:R_0805_HandSoldering, B.Cu at (56.8, 49.5)
- added R5: 100k, Resistors_SMD:R_0805_HandSoldering, B.Cu at (56.8, 51.5)
- added SW1: SW_PUSH, Cartel:c&k_PTS645SH50SMTR92_LFS, B.Cu at (33.3, 85.7)
- added U1: nRF24L01+, Cartel:nRF24L01+_SMD, B.Cu at (14.8, 57.2)
- added U2: MCP1700T-3002E/TT, TO_SOT_Packages_SMD:SOT-23_Handsoldering, B.Cu at (62.0, 41.2)
- moved D12 38.1 mm to (195.3, 47.1)
- moved D4 19.1 mm to (81.0, 47.1)
- moved D5 19.0 mm to (100.0, 47.1)
- moved D26 16.7 mm to (207.2, 66.2)
- moved D11 16.7 mm to (197.6, 47.1)
- moved D16 5.26 mm to (9.53, 71.4)
- moved D1 2.38 mm to (7.14, 44.7)
- moved D2 2.38 mm to (40.5, 44.7)
- moved D3 2.38 mm to (45.2, 44.7)
- moved D10 2.38 mm to (192.9, 47.1)
- moved D17 2.38 mm to (54.8, 66.2)
- moved D25 2.38 mm to (202.4, 66.2)
- moved D66 1.01 mm to (288.4, 124.3)
- moved D27 1.00 mm to (241.5, 66.2)
- moved D28 0.77 mm to (244.5, 66.2)
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Connections:
- net Net-(D1-Pad1) renamed /ROW0
- net Net-(D16-Pad1) renamed /ROW1
- net Net-(D30-Pad1) renamed /ROW2
- net Net-(D44-Pad1) renamed /ROW3
- net Net-(D58-Pad1) renamed /ROW4
- net Net-(K10-Pad1) renamed /COL9
- net Net-(K11-Pad1) renamed /COL10
- net Net-(K18-Pad1) renamed /COL2
- net Net-(K19-Pad1) renamed /COL3
- net Net-(K2-Pad1) renamed /COL1
- net Net-(K20-Pad1) renamed /COL4
- net Net-(K21-Pad1) renamed /COL5
- net Net-(K22-Pad1) renamed /COL6
- net Net-(K23-Pad1) renamed /COL7
- net Net-(K24-Pad1) renamed /COL8
- K1 pad 1: Net-(K1-Pad1) -> /COL0
- K12 pad 1: Net-(K12-Pad1) -> /COL11
- K13 pad 1: Net-(K13-Pad1) -> /COL12
- K14 pad 1: Net-(K14-Pad1) -> /COL14
- K15 pad 1: Net-(K15-Pad1) -> /COL13
- K16 pad 1: Net-(K14-Pad1) -> /COL14
- K17 pad 1: Net-(K1-Pad1) -> /COL0
- K27 pad 1: Net-(K12-Pad1) -> /COL11
- K28 pad 1: Net-(K13-Pad1) -> /COL12
- K29 pad 1: Net-(K15-Pad1) -> /COL13
- K30 pad 1: Net-(K14-Pad1) -> /COL14
- K31 pad 1: Net-(K1-Pad1) -> /COL0
- K41 pad 1: Net-(K12-Pad1) -> /COL11
- K42 pad 1: Net-(K13-Pad1) -> /COL12
- K43 pad 1: Net-(K14-Pad1) -> /COL14
- K44 pad 1: Net-(K1-Pad1) -> Net-(D30-Pad2)
- K44 pad 2: Net-(D30-Pad2) -> /COL0
- K45 pad 1: Net-(K15-Pad1) -> /COL13
- K46 pad 1: Net-(K46-Pad1) -> /COL14
- K47 pad 1: Net-(K13-Pad1) -> Net-(D55-Pad2)
- K47 pad 2: Net-(D55-Pad2) -> /COL12
- K48 pad 1: Net-(K15-Pad1) -> /COL13
- K49 pad 1: Net-(K1-Pad1) -> /COL0
- K59 pad 1: Net-(K15-Pad1) -> Net-(D56-Pad2)
- K59 pad 2: Net-(D56-Pad2) -> /COL13
- K60 pad 1: Net-(K14-Pad1) -> /COL14
- K61 pad 1: Net-(K1-Pad1) -> Net-(D44-Pad2)
- K61 pad 2: Net-(D44-Pad2) -> /COL0
- K63 pad 1: Net-(K15-Pad1) -> /COL13
- K64 pad 1: Net-(K14-Pad1) -> Net-(D57-Pad2)
- K64 pad 2: Net-(D57-Pad2) -> /COL14
- K65 pad 1: Net-(K13-Pad1) -> /COL12
- K66 pad 1: Net-(K15-Pad1) -> /COL13
- K67 pad 1: Net-(K14-Pad1) -> /COL14
- K68 pad 1: Net-(K1-Pad1) -> /COL0
- K73 pad 1: Net-(K12-Pad1) -> /COL11
- K74 pad 1: Net-(K15-Pad1) -> /COL13
- K75 pad 1: Net-(K14-Pad1) -> /COL14
- K76 pad 1: Net-(K1-Pad1) -> /COL0
- K80 pad 1: Net-(K12-Pad1) -> /COL11
- K81 pad 1: Net-(K15-Pad1) -> /COL13
- K82 pad 1: Net-(K14-Pad1) -> /COL14
- K84 pad 1: Net-(K12-Pad1) -> Net-(D63-Pad2)
- K84 pad 2: Net-(D63-Pad2) -> /COL11
- K85 pad 1: Net-(K13-Pad1) -> /COL12
- K86 pad 1: Net-(K15-Pad1) -> Net-(D65-Pad2)
- K86 pad 2: Net-(D65-Pad2) -> /COL13
- K87 pad 1: Net-(K14-Pad1) -> /COL14
Routing:
- net /COL14: track 0.00 -> 384.6 mm
- net /COL13: track 0.00 -> 347.7 mm
- net /COL12: track 0.00 -> 290.5 mm
- net /ROW3: track 0.00 -> 279.7 mm
- net /COL11: track 0.00 -> 279.5 mm
- net GND: track 0.00 -> 278.5 mm, vias 0 -> 2
- net /ROW4: track 0.00 -> 266.1 mm
- net /COL10: track 0.00 -> 245.8 mm
- net /ROW2: track 0.00 -> 227.2 mm
- net /ROW1: track 0.00 -> 210.2 mm
- net /COL9: track 0.00 -> 206.0 mm
- net /COL8: track 0.00 -> 187.9 mm
- net /COL6: track 0.00 -> 182.8 mm
- net /COL7: track 0.00 -> 169.4 mm
- net Net-(BT1-Pad1): track 0.00 -> 151.8 mm
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Other:
- net class Power added: clearance 0.2, trace_width 0.4, via_dia 0.6, via_drill 0.4
- board text added: "PDI"

Commit message: Finished PCB functionality
Parts:
- added D68: 1N4148, Diodes_SMD:D_SOD-323_HandSoldering, B.Cu at (111.9, 125.0)
- added D69: 1N4148, Diodes_SMD:D_SOD-323_HandSoldering, B.Cu at (159.5, 125.0)
- added J1: USB_mini_micro_B, keyboard_parts:USB_miniB_hirose_5S8, B.Cu at (23.8, 45.0)
- added K88: KEYSW, MXAlps:MX-2.75U-ReversedStabilizer-NoLED, F.Cu at (102.4, 123.8)
- added K89: KEYSW, MXAlps:MX-1.25U-NoLED, F.Cu at (140.5, 123.8)
- added K90: KEYSW, MXAlps:MX-2.25U-ReversedStabilizer-NoLED, F.Cu at (173.8, 123.8)
- added K91: KEYSW, MXAlps:MX-2.25U-ReversedStabilizer-NoLED, F.Cu at (97.6, 123.8)
- added K92: KEYSW, MXAlps:MX-1.25U-NoLED, F.Cu at (131.0, 123.8)
- added K93: KEYSW, MXAlps:MX-2.75U-ReversedStabilizer-NoLED, F.Cu at (169.1, 123.8)
- added K94: KEYSW, MXAlps:MX-2.25U-ReversedStabilizer-NoLED, F.Cu at (102.4, 123.8)
- added K95: KEYSW, MXAlps:MX-2U-ReversedStabilizers-NoLED, F.Cu at (142.9, 123.8)
- added K96: KEYSW, MXAlps:MX-2.75U-ReversedStabilizer-NoLED, F.Cu at (188.1, 123.8)
- D1, D10, D11, D12, D13, D14, D15, D16, D17, D18, D19, D2, D20, D21, D22, D23, D24, D25, D26, D27, D28, D29, D3, D30, D31, D32, D33, D34, D35, D36, D37, D38, D39, D4, D40, D41, D42, D43, D44, D45, D46, D47, D48, D49, D5, D50, D51, D52, D53, D54, D55, D56, D57, D58, D59, D6, D60, D61, D62, D63, D64, D65, D66, D7, D8, D9: footprint Cartel:combo_diode -> Diodes_SMD:D_SOD-323_HandSoldering
- moved D64 54.8 mm to (269.1, 125.0)
- moved D12 40.5 mm to (235.7, 48.8)
- moved D62 26.2 mm to (214.3, 125.0)
- moved D16 19.1 mm to (28.5, 73.2)
- moved D65 4.39 mm to (265.0, 125.0)
- moved U2 3.20 mm to (62.0, 44.5)
- moved C5 2.95 mm to (62.5, 47.2)
- moved D14 2.93 mm to (254.8, 48.8)
- moved D15 2.93 mm to (252.4, 48.8)
- moved D17 2.93 mm to (52.4, 67.9)
- moved D26 2.93 mm to (204.8, 67.9)
- moved D67 2.70 mm to (62.0, 50.0)
- moved D27 2.14 mm to (242.9, 67.9)
- moved R2 2.09 mm to (24.5, 48.7)
- moved R3 2.01 mm to (26.2, 48.7)
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Connections:
- IC1 pad 20: /ROW4 -> /ROW1
- IC1 pad 21: /ROW3 -> /ROW4
- IC1 pad 22: /ROW2 -> /ROW3
- IC1 pad 23: /ROW1 -> /ROW2
Routing:
- net /ROW0: track 131.1 -> 277.1 mm, vias 1 -> 6
- net /ROW4: track 266.1 -> 351.7 mm, vias 0 -> 2
- net GND: track 278.5 -> 359.8 mm, vias 2 -> 4
- net /ROW3: track 279.7 -> 350.8 mm, vias 0 -> 2
- net /ROW1: track 210.2 -> 272.9 mm, vias 0 -> 3
- net /ROW2: track 227.2 -> 279.9 mm, vias 0 -> 2
- net +5V: track 9.84 -> 58.2 mm
- net Net-(D15-Pad2): track 0.00 -> 39.7 mm
- net Net-(D69-Pad2): track 0.00 -> 36.8 mm
- net /COL8: track 187.9 -> 223.4 mm
- net Net-(D61-Pad2): track 13.0 -> 43.6 mm
- net Net-(D68-Pad2): track 0.00 -> 25.0 mm
- net Net-(D44-Pad2): track 0.00 -> 23.8 mm
- net /COL4: track 131.5 -> 154.7 mm
- net Net-(D30-Pad2): track 0.00 -> 22.5 mm
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Other:
- board text added: "Diodes placed at 1.2mm offset"
- board text removed: "Diodes placed at -0.5mm offset"

Commit message: Add fuse
Parts:
- added F1: PPTC, Fuse_Holders_and_Fuses:Fuse_SMD1206_HandSoldering, B.Cu at (42.8, 41.8)
Connections:
- J1 pad 1: +5V -> Net-(F1-Pad1)
Routing:
- net +5V: track 58.2 -> 26.4 mm
- net Net-(F1-Pad1): track 0.00 -> 28.8 mm
- net Net-(D3-Pad2): track 15.6 -> 11.4 mm
- net /ROW0: track 277.1 -> 275.9 mm
- net Net-(D2-Pad2): track 6.16 -> 5.50 mm

Commit message: Begin decorating
Parts:
- added G***: LOGO, logo:amtra5-15.2mm, F.Cu at (182.6, 92.9)
- added G***: LOGO, logo:cartel-7.8mm, F.Cu at (224.6, 93.7)
Other:
- board text added: "amtra5"
- board text added: "rf60"
- board text added: "wireless keyboard"
