File: 60.kicad_pcb (KiCad board)
At the start: 2 copper layers, 285 x 94.6 mm, 186 parts, among them IC1 ATXMEGA32A4U-A, J1 USB_mini_micro_B, K1 KEYSW, K10 KEYSW, K11 KEYSW, K12 KEYSW, K13 KEYSW, K14 KEYSW, K15 KEYSW, K16 KEYSW, K17 KEYSW, K18 KEYSW, K19 KEYSW, K2 KEYSW, K20 KEYSW, K21 KEYSW, K22 KEYSW, K23 KEYSW, K24 KEYSW, K25 KEYSW, K26 KEYSW, K27 KEYSW, K28 KEYSW, K29 KEYSW, K3 KEYSW, K30 KEYSW, K31 KEYSW, K32 KEYSW, K33 KEYSW, K34 KEYSW, K35 KEYSW, K36 KEYSW, K37 KEYSW, K38 KEYSW, K39 KEYSW, K4 KEYSW, K40 KEYSW, K41 KEYSW, K42 KEYSW, K43 KEYSW, K44 KEYSW, K45 KEYSW, K46 KEYSW, K47 KEYSW, K48 KEYSW, K49 KEYSW, K5 KEYSW, K50 KEYSW, K51 KEYSW, K52 KEYSW, K53 KEYSW, K54 KEYSW, K55 KEYSW, K56 KEYSW, K57 KEYSW, K58 KEYSW, K59 KEYSW, K6 KEYSW, K60 KEYSW, K61 KEYSW, K62 KEYSW, K63 KEYSW, K64 KEYSW, K65 KEYSW, K66 KEYSW, K67 KEYSW, K68 KEYSW, K69 KEYSW, K7 KEYSW, K70 KEYSW, K71 KEYSW, K72 KEYSW, K73 KEYSW, K74 KEYSW, K75 KEYSW, K76 KEYSW, K77 KEYSW, K78 KEYSW, K79 KEYSW, K8 KEYSW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

Commit message: Prototype 1
Parts:
- removed F1: PPTC, Fuse_Holders_and_Fuses:Fuse_SMD1206_HandSoldering
- removed R2, R3: 22, Resistors_SMD:R_0805_HandSoldering
- added C6: 0.1uF, Capacitors_SMD:C_0805_HandSoldering, B.Cu at (39.0, 90.0)
- added SJ1: SOLDER_JUMPER, keyboard_parts:SOLDER_JUMPER_2, B.Cu at (208.5, 53.8)
- added SW2: POWER, Pin_Headers:Pin_Header_Straight_1x02_Pitch2.54mm, B.Cu at (207.0, 57.0)
- BT1: footprint Battery_Holders:Keystone_1058_1x2032-CoinCell -> lib:CR2032_BK-913
- D67: value D_Schottky_x2_KCom_AAK -> BAT54C-7-F
- P1: value CONN_01X01 -> TC2030-MCP-NL; footprint Connectors_TestPoints:Test_Point_Pad_2.0x2.0mm -> Tag-Connect:TC2030-MCP-NL
- SW1: footprint Cartel:c&k_PTS645SH50SMTR92_LFS -> Buttons_Switches_SMD:SW_SPST_TL3342
- moved P1 37.5 mm to (39.0, 87.5), turned to 90 degrees
- moved D1 11.8 mm to (18.2, 50.0), turned to 180 degrees
- moved BT1 1.77 mm to (224.0, 58.8), turned to 180 degrees
Connections:
- D67 pad 2: Net-(BT1-Pad1) -> Net-(D67-Pad2)
- IC1 pad 34: Net-(IC1-Pad34) -> /PDI
- IC1 pad 35: Net-(IC1-Pad35) -> /PDI_CLK
- J1 pad 1: Net-(F1-Pad1) -> +5V
- J1 pad 2: Net-(J1-Pad2) -> /D-
- J1 pad 3: Net-(J1-Pad3) -> /D+
- J1 pad 6: GND -> Net-(J1-Pad6)
- P1 pad 1: Net-(IC1-Pad34) -> Net-(P1-Pad1)
- R1 pad 2: Net-(IC1-Pad35) -> /PDI_CLK
- SW1 pad 2: Net-(IC1-Pad35) -> /PDI_CLK
- U1 pad 3: Net-(U1-Pad3) -> Net-(IC1-Pad25)
- U1 pad 8: Net-(U1-Pad8) -> Net-(IC1-Pad13)
Routing:
- net Net-(D67-Pad2): track 0.00 -> 150.7 mm
- net Net-(BT1-Pad1): track 150.7 -> 40.7 mm
- net /PDI: track 0.00 -> 49.2 mm, vias 0 -> 2
- net /PDI_CLK: track 0.00 -> 48.7 mm, vias 0 -> 2
- net Net-(IC1-Pad35): track 46.5 -> 0.00 mm, vias 2 -> 0
- net +5V: track 26.4 -> 58.4 mm, vias 2 -> 4
- net Net-(F1-Pad1): track 28.8 -> 0.00 mm
- net +3V3: track 94.4 -> 118.5 mm
- net Net-(IC1-Pad25): track 0.00 -> 21.7 mm, vias 0 -> 4
- net /ROW0: track 275.9 -> 262.1 mm
- net Net-(IC1-Pad13): track 0.00 -> 12.8 mm
- net Net-(D1-Pad2): track 13.1 -> 6.96 mm
- net /D+: track 16.6 -> 22.7 mm
- net Net-(J1-Pad3): track 4.17 -> 0.00 mm
- net /D-: track 18.4 -> 22.5 mm
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- added copper zone on B.Cu, net GND
- added copper zone on F.Cu, net GND

Commit message: Prototype 1 fix
Fix tag connect and added airi
Parts:
- added G***: LOGO, lib:airi-silk-5mm, B.Cu at (33.3, 92.9)
- C6: value 0.1uF -> 0.1u
- P1: value TC2030-MCP-NL -> TC2030-IDC; footprint Tag-Connect:TC2030-MCP-NL -> Tag-Connect:TC2030-NL_SMALL
- moved C6 11.5 mm to (40.0, 78.5)
- moved P1 2.50 mm to (39.0, 85.0)
Connections:
- P1 pad 1: Net-(P1-Pad1) -> /PDI
- P1 pad 3: GND -> Net-(P1-Pad3)
- P1 pad 4: /PDI -> Net-(P1-Pad4)
- P1 pad 6: Net-(P1-Pad6) -> GND
Routing:
- net +3V3: track 118.5 -> 110.5 mm
- net /PDI: track 49.2 -> 54.8 mm
- net GND: track 360.3 -> 360.1 mm, vias 10 -> 9

Commit message: Prototype 1 last fix
Parts:
- moved BT1 2.50 mm to (224.0, 56.2), turned to 0 degrees
Routing:
- net GND: track 360.1 -> 374.2 mm, vias 9 -> 11
- net Net-(BT1-Pad1): track 40.7 -> 33.2 mm
Changed lines of the file:
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@@
     (thickness 1.6)
     (drawings 31)
-    (tracks 1246)
+    (tracks 1245)
     (zones 0)
     (modules 187)
@@
   )
   (module lib:CR2032_BK-913 (layer B.Cu)
-    (at 224 58.75 180)
+    (at 224 56.25)
     (zone_connect 2)
-    (fp_text reference BT1 (at 0 -4.8 180) (layer B.SilkS)
+    (fp_text reference BT1 (at 0 -4.8) (layer B.SilkS)
       (effects (font (size 1 1) (thickness 0.15)) (justify mirror))
     )
-    (fp_text value Battery (at -0.5 -7 180) (layer B.Fab)
+    (fp_text value Battery (at -0.5 -7) (layer B.Fab)
       (effects (font (size 1 1) (thickness 0.15)) (justify mirror))
     )
@@
     (fp_line (start 11.5 -11.5) (end 11.5 11.5) (layer B.CrtYd) (width 0.1))
     (fp_line (start 11.5 11.5) (end -11.5 11.5) (layer B.CrtYd) (width 0.1))
-    (pad 1 thru_hole circle (at 10.8 0 180) (size 3 3) (drill 2) (layers *.Cu *.Paste *.Mask)
+    (pad 1 thru_hole circle (at 10.8 0) (size 3 3) (drill 2) (layers *.Cu *.Paste *.Mask)
       (net 67 "Net-(BT1-Pad1)") (zone_connect 2))
-    (pad 2 smd rect (at 0 0 180) (size 7 7) (layers B.Cu B.Mask)
+    (pad 2 smd rect (at 0 0) (size 7 7) (layers B.Cu B.Mask)
       (net 68 GND) (zone_connect 2))
-    (pad 1 thru_hole circle (at -10.8 0 180) (size 3 3) (drill 2) (layers *.Cu *.Paste *.Mask)
+    (pad 1 thru_hole circle (at -10.8 0) (size 3 3) (drill 2) (layers *.Cu *.Paste *.Mask)
       (net 67 "Net-(BT1-Pad1)") (zone_connect 2))
   )
@@
   (segment (start 268 116.95) (end 247.7625 116.95) (width 0.25) (layer B.Cu) (net 66))
   (segment (start 269.08125 118.03125) (end 268 116.95) (width 0.25) (layer B.Cu) (net 66))
-  (segment (start 208.5 54.15) (end 211.9 54.15) (width 0.4) (layer B.Cu) (net 67))
-  (segment (start 213.2 55.45) (end 213.2 58.75) (width 0.4) (layer B.Cu) (net 67))
-  (segment (start 211.9 54.15) (end 213.2 55.45) (width 0.4) (layer B.Cu) (net 67))
-  (segment (start 213.2 58.75) (end 211.29 58.75) (width 0.4) (layer B.Cu) (net 67))
-  (segment (start 211.29 58.75) (end 209.54 57) (width 0.4) (layer B.Cu) (net 67))
-  (segment (start 228.75 53.5) (end 232.75 53.5) (width 0.4) (layer B.Cu) (net 67))
-  (segment (start 213.2 58.75) (end 217.41 54.54) (width 0.4) (layer B.Cu) (net 67))
-  (segment (start 218.45 53.5) (end 217.41 54.54) (width 0.4) (layer B.Cu) (net 67))
-  (segment (start 233.75 54.5) (end 234.8 55.55) (width 0.4) (layer B.Cu) (net 67))
-  (segment (start 234.8 55.55) (end 234.8 58.75) (width 0.4) (layer B.Cu) (net 67))
-  (segment (start 219.25 53.5) (end 228.75 53.5) (width 0.4) (layer B.Cu) (net 67))
-  (segment (start 219.25 53.5) (end 218.45 53.5) (width 0.4) (layer B.Cu) (net 67))
-  (segment (start 232.75 53.5) (end 233.75 54.5) (width 0.4) (layer B.Cu) (net 67))
+  (segment (start 213.2 56.25) (end 213.25 56.25) (width 0.4) (layer B.Cu) (net 67))
+  (segment (start 213.25 56.25) (end 218.5 51) (width 0.4) (layer B.Cu) (net 67))
+  (segment (start 229.55 51) (end 234.8 56.25) (width 0.4) (layer B.Cu) (net 67))
+  (segment (start 218.5 51) (end 229.55 51) (width 0.4) (layer B.Cu) (net 67))
+  (segment (start 213.2 56.25) (end 210.29 56.25) (width 0.4) (layer B.Cu) (net 67))
+  (segment (start 210.29 56.25) (end 209.54 57) (width 0.4) (layer B.Cu) (net 67))
+  (segment (start 209.54 57) (end 209.54 55.19) (width 0.4) (layer B.Cu) (net 67))
+  (segment (start 209.54 55.19) (end 208.5 54.15) (width 0.4) (layer B.Cu) (net 67))
+  (segment (start 224 56.25) (end 217.5 56.25) (width 0.4) (layer B.Cu) (net 68))
+  (via (at 217.5 56.25) (size 0.6) (drill 0.4) (layers F.Cu B.Cu) (net 68))
+  (segment (start 224 56.25) (end 230.5 56.25) (width 0.4) (layer B.Cu) (net 68))
+  (via (at 230.5 56.25) (size 0.6) (drill 0.4) (layers F.Cu B.Cu) (net 68))
+  (segment (start 215.25 61) (end 219.25 61) (width 0.4) (layer B.Cu) (net 68))
+  (segment (start 204.75 53) (end 203.75 52) (width 0.4) (layer B.Cu) (net 68))
+  (segment (start 203.75 52) (end 201 52) (width 0.4) (layer B.Cu) (net 68))
+  (segment (start 207.25 61) (end 205.75 61) (width 0.4) (layer B.Cu) (net 68))
+  (segment (start 207.25 61) (end 215.25 61) (width 0.4) (layer B.Cu) (net 68))
+  (segment (start 205.75 61) (end 204.75 60) (width 0.4) (layer B.Cu) (net 68))
+  (segment (start 62.25 51.95) (end 62.3 52) (width 0.4) (layer B.Cu) (net 68))
+  (segment (start 201 52) (end 63 52) (width 0.4) (layer B.Cu) (net 68))
+  (segment (start 63 52) (end 62.3 52) (width 0.4) (layer B.Cu) (net 68))
+  (segment (start 204.75 60) (end 204.75 53) (width 0.4) (layer B.Cu) (net 68))
+  (segment (start 219.25 61) (end 224 56.25) (width 0.4) (layer B.Cu) (net 68))
   (segment (start 34.25 77.5) (end 34.25 76.25) (width 0.4) (layer F.Cu) (net 68))
   (segment (start 34.75 78) (end 34.25 77.5) (width 0.4) (layer F.Cu) (net 68))
@@
   (segment (start 40.5 80) (end 39.5 80) (width 0.4) (layer B.Cu) (net 68))
   (segment (start 41.25 80.75) (end 40.5 80) (width 0.4) (layer B.Cu) (net 68))
-  (segment (start 204.75 60) (end 204.75 53) (width 0.4) (layer B.Cu) (net 68))
-  (segment (start 63 52) (end 62.3 52) (width 0.4) (layer B.Cu) (net 68))
-  (segment (start 201 52) (end 63 52) (width 0.4) (layer B.Cu) (net 68))
-  (segment (start 62.25 51.95) (end 62.3 52) (width 0.4) (layer B.Cu) (net 68))
-  (segment (start 205.75 61) (end 204.75 60) (width 0.4) (layer B.Cu) (net 68))
-  (segment (start 215.25 61) (end 221.75 61) (width 0.4) (layer B.Cu) (net 68))
-  (segment (start 207.25 61) (end 215.25 61) (width 0.4) (layer B.Cu) (net 68))
-  (segment (start 207.25 61) (end 205.75 61) (width 0.4) (layer B.Cu) (net 68))
-  (segment (start 203.75 52) (end 201 52) (width 0.4) (layer B.Cu) (net 68))
-  (segment (start 204.75 53) (end 203.75 52) (width 0.4) (layer B.Cu) (net 68))
   (segment (start 60.5 51.95) (end 60.5 51.25) (width 0.4) (layer B.Cu) (net 68))
   (via (at 60.25 59) (size 0.6) (drill 0.4) (layers F.Cu B.Cu) (net 68))
@@
   (segment (start 35.75 74.25) (end 35.75 69.25) (width 0.4) (layer B.Cu) (net 68))
   (segment (start 31.0875 82.225) (end 31.4375 82.575) (width 0.4) (layer B.Cu) (net 68))
-  (segment (start 221.75 61) (end 224 58.75) (width 0.4) (layer B.Cu) (net 68))
   (segment (start 23.75 54.12) (end 22.92 54.12) (width 0.4) (layer B.Cu) (net 68))
   (segment (start 35.75 69.25) (end 36.75 69.25) (width 0.4) (layer B.Cu) (net 68))
